Commit message: Add four groundtruth imu on the center of each arm.

File: rotors_description/urdf/component_snippets.xacro (robot description, xacro)
@@ -748,5 +748,5 @@
       parent_link="${namespace}/vi_sensor_link"
       imu_topic="imu"
-      mass_imu_sensor="0.015"
+      mass_imu_sensor="0.0000015"
       gyroscope_noise_density="0.0003394"
       gyroscope_random_walk="0.000038785"
@@ -818,15 +818,83 @@
       parent_link="${parent_link}"
       imu_topic="imu"
-      mass_imu_sensor="0.015"
-      gyroscope_noise_density="0.0003394"
-      gyroscope_random_walk="0.000038785"
+      mass_imu_sensor="0.00001"
+      gyroscope_noise_density="0.0"
+      gyroscope_random_walk="0.0"
       gyroscope_bias_correlation_time="1000.0"
-      gyroscope_turn_on_bias_sigma="0.0087"
-      accelerometer_noise_density="0.004"
-      accelerometer_random_walk="0.006"
+      gyroscope_turn_on_bias_sigma="0.0"
+      accelerometer_noise_density="0.0"
+      accelerometer_random_walk="0.0"
       accelerometer_bias_correlation_time="300.0"
-      accelerometer_turn_on_bias_sigma="0.1960">
+      accelerometer_turn_on_bias_sigma="0.0">
       <inertia ixx="0.00001" ixy="0.0" ixz="0.0" iyy="0.00001" iyz="0.0" izz="0.00001" />
       <origin xyz="0 0 0" rpy="0 0 0" />
+    </xacro:imu_plugin_macro>
+    <xacro:imu_plugin_macro
+      namespace="${namespace}"
+      imu_suffix="1"
+      parent_link="${parent_link}"
+      imu_topic="imu1"
+      mass_imu_sensor="0.00001"
+      gyroscope_noise_density="0.0"
+      gyroscope_random_walk="0.0"
+      gyroscope_bias_correlation_time="1000.0"
+      gyroscope_turn_on_bias_sigma="0.0"
+      accelerometer_noise_density="0.0"
+      accelerometer_random_walk="0.0"
+      accelerometer_bias_correlation_time="300.0"
+      accelerometer_turn_on_bias_sigma="0.0">
+      <inertia ixx="0.00001" ixy="0.0" ixz="0.0" iyy="0.00001" iyz="0.0" izz="0.00001" />
+      <origin xyz="0.1 0 0" rpy="0 0 0" />
+    </xacro:imu_plugin_macro>
+    <xacro:imu_plugin_macro
+      namespace="${namespace}"
+      imu_suffix="2"
+      parent_link="${parent_link}"
+      imu_topic="imu2"
+      mass_imu_sensor="0.00001"
+      gyroscope_noise_density="0.0"
+      gyroscope_random_walk="0.0"
+      gyroscope_bias_correlation_time="1000.0"
+      gyroscope_turn_on_bias_sigma="0.0"
+      accelerometer_noise_density="0.0"
+      accelerometer_random_walk="0.0"
+      accelerometer_bias_correlation_time="300.0"
+      accelerometer_turn_on_bias_sigma="0.0">
+      <inertia ixx="0.00001" ixy="0.0" ixz="0.0" iyy="0.00001" iyz="0.0" izz="0.00001" />
+      <origin xyz="0 0.1 0" rpy="0 0 0" />
+    </xacro:imu_plugin_macro>
+    <xacro:imu_plugin_macro
+      namespace="${namespace}"
+      imu_suffix="3"
+      parent_link="${parent_link}"
+      imu_topic="imu3"
+      mass_imu_sensor="0.00001"
+      gyroscope_noise_density="0.0"
+      gyroscope_random_walk="0.0"
+      gyroscope_bias_correlation_time="1000.0"
+      gyroscope_turn_on_bias_sigma="0.0"
+      accelerometer_noise_density="0.0"
+      accelerometer_random_walk="0.0"
+      accelerometer_bias_correlation_time="300.0"
+      accelerometer_turn_on_bias_sigma="0.0">
+      <inertia ixx="0.00001" ixy="0.0" ixz="0.0" iyy="0.00001" iyz="0.0" izz="0.00001" />
+      <origin xyz="-0.1 0 0" rpy="0 0 0" />
+    </xacro:imu_plugin_macro>
+    <xacro:imu_plugin_macro
+      namespace="${namespace}"
+      imu_suffix="4"
+      parent_link="${parent_link}"
+      imu_topic="imu4"
+      mass_imu_sensor="0.00001"
+      gyroscope_noise_density="0.0"
+      gyroscope_random_walk="0.0"
+      gyroscope_bias_correlation_time="1000.0"
+      gyroscope_turn_on_bias_sigma="0.0"
+      accelerometer_noise_density="0.0"
+      accelerometer_random_walk="0.0"
+      accelerometer_bias_correlation_time="300.0"
+      accelerometer_turn_on_bias_sigma="0.0">
+      <inertia ixx="0.00001" ixy="0.0" ixz="0.0" iyy="0.00001" iyz="0.0" izz="0.00001" />
+      <origin xyz="0 -0.1 0" rpy="0 0 0" />
     </xacro:imu_plugin_macro>
   </xacro:macro>
